File: electronics/led_board_stack_light/led_board.sch (KiCad schematic (older format))
At the start: 14 parts, among them J1 CONN_01X02, J2 CONN_01X01, P1 OSHW, P2 Slot, P3 Slot, P4 Slot

Commit message: Minor changes, but wire in outliner script
Parts:
- D1, D2, D3, D4, D5, D6, R1: MFN (none) -> Lite-On Inc.; MPN (none) -> LTW-670DS
Other:
- note added: "+12V in, out to next light"
- note added: "Switched GND"
- note added: "White 3528 (PLCC-2) size LEDs,\n12V in, 3.4Vf gives 61mW\ndissipated in each resistor."
- note removed: "White 3528 (PLCC-2) size LEDs,\n12V in, 3.4Vf gives 61mW"
- moved on the sheet: J1
Changed lines of the file:
@@
 Date ""
 Rev ""
-Comp ""
-Comment1 ""
+Comp "(c) Google LLC"
+Comment1 "CC-BY 4.0 International"
 Comment2 ""
 Comment3 ""
@@
 F 2 "LEDs:LED_PLCC-2" H 6000 3000 50  0001 C CNN
 F 3 "" H 6000 3000 50  0001 C CNN
+F 4 "LTW-670DS" H 6000 3000 60  0001 C CNN "MPN"
+F 5 "Lite-On Inc." H 6000 3000 60  0001 C CNN "MFN"
 	1    6000 3000
 	0    -1   -1   0
@@
 F 2 "LEDs:LED_PLCC-2" H 6000 3400 50  0001 C CNN
 F 3 "" H 6000 3400 50  0001 C CNN
+F 4 "LTW-670DS" H 6000 3000 60  0001 C CNN "MPN"
+F 5 "Lite-On Inc." H 6000 3000 60  0001 C CNN "MFN"
 	1    6000 3400
 	0    -1   -1   0
@@
 F 2 "LEDs:LED_PLCC-2" H 6000 3800 50  0001 C CNN
 F 3 "" H 6000 3800 50  0001 C CNN
+F 4 "LTW-670DS" H 6000 3000 60  0001 C CNN "MPN"
+F 5 "Lite-On Inc." H 6000 3000 60  0001 C CNN "MFN"
 	1    6000 3800
 	0    -1   -1   0
@@
 F 2 "Resistors_SMD:R_0805" V 5930 4300 50  0001 C CNN
 F 3 "" H 6000 4300 50  0001 C CNN
+F 4 "LTW-670DS" H 6000 3000 60  0001 C CNN "MPN"
+F 5 "Lite-On Inc." H 6000 3000 60  0001 C CNN "MFN"
 	1    6000 4300
 	1    0    0    -1
@@
 F 2 "LEDs:LED_PLCC-2" H 6400 3000 50  0001 C CNN
 F 3 "" H 6400 3000 50  0001 C CNN
+F 4 "LTW-670DS" H 6000 3000 60  0001 C CNN "MPN"
+F 5 "Lite-On Inc." H 6000 3000 60  0001 C CNN "MFN"
 	1    6400 3000
 	0    -1   -1   0
@@
 F 2 "LEDs:LED_PLCC-2" H 6400 3400 50  0001 C CNN
 F 3 "" H 6400 3400 50  0001 C CNN
+F 4 "LTW-670DS" H 6000 3000 60  0001 C CNN "MPN"
+F 5 "Lite-On Inc." H 6000 3000 60  0001 C CNN "MFN"
 	1    6400 3400
 	0    -1   -1   0
@@
 F 2 "LEDs:LED_PLCC-2" H 6400 3800 50  0001 C CNN
 F 3 "" H 6400 3800 50  0001 C CNN
+F 4 "LTW-670DS" H 6000 3000 60  0001 C CNN "MPN"
+F 5 "Lite-On Inc." H 6000 3000 60  0001 C CNN "MFN"
 	1    6400 3800
 	0    -1   -1   0
@@
 $EndComp
 Wire Wire Line
-	4900 2800 6400 2800
-Wire Wire Line
-	6400 4550 5550 4550
-Text Notes 5700 2600 0    60   ~ 0
-White 3528 (PLCC-2) size LEDs,\n12V in, 3.4Vf gives 61mW
+	4950 2800 5050 2800
+Wire Wire Line
+	5050 2800 6000 2800
+Wire Wire Line
+	6000 2800 6400 2800
+Wire Wire Line
+	6400 4550 6000 4550
+Wire Wire Line
+	6000 4550 5550 4550
+Text Notes 6700 4450 0    60   ~ 0
+White 3528 (PLCC-2) size LEDs,\n12V in, 3.4Vf gives 61mW\ndissipated in each resistor.
 $Comp
 L SYMBOL P2
@@
 L CONN_01X02 J1
 U 1 1 5A7E0D6B
-P 4950 2550
-F 0 "J1" H 4950 2700 50  0000 C CNN
-F 1 "CONN_01X02" V 5050 2550 50  0000 C CNN
-F 2 "Pin_Headers:Pin_Header_Straight_1x02_Pitch2.54mm" H 4950 2550 50  0001 C CNN
-F 3 "" H 4950 2550 50  0001 C CNN
-	1    4950 2550
+P 5000 2550
+F 0 "J1" H 5000 2700 50  0000 C CNN
+F 1 "CONN_01X02" V 5100 2550 50  0000 C CNN
+F 2 "Pin_Headers:Pin_Header_Straight_1x02_Pitch2.54mm" H 5000 2550 50  0001 C CNN
+F 3 "" H 5000 2550 50  0001 C CNN
+	1    5000 2550
 	0    -1   -1   0
 $EndComp
@@
 	5000 2900 5000 2950
 Wire Wire Line
-	5000 2800 5000 2750
-Wire Wire Line
-	4900 2800 4900 2750
-Connection ~ 5000 2800
+	5050 2800 5050 2750
+Wire Wire Line
+	4950 2800 4950 2750
+Connection ~ 5050 2800
+Text Notes 4450 2300 0    60   ~ 0
++12V in, out to next light
+Text Notes 4700 3450 0    60   ~ 0
+Switched GND
 $EndSCHEMATC
