File: electronics/led_board_stack_light/led_board.sch (KiCad schematic (older format))
At the start: 14 parts, among them J1 CONN_01X02, J2 CONN_01X01, P1 OSHW, P2 Slot, P3 Slot, P4 Slot

Commit message: Minor updates on recent boards
Parts:
- added P5: US0119, OSHWA_Certification_Mark:OSHW_Mono_0.15_Scale, symbol SYMBOL
Changed lines of the file:
@@
 encoding utf-8
 Sheet 1 1
-Title ""
+Title "Machine Status Indicator"
 Date ""
 Rev ""
@@
 Comment1 ""
 Comment2 ""
-Comment3 ""
-Comment4 ""
+Comment3 "(c) Google LLC"
+Comment4 "CC-BY 4.0 International"
 $EndDescr
 $Comp
@@
 	4900 2800 4900 2750
 Connection ~ 5000 2800
+$Comp
+L SYMBOL P5
+U 1 1 5AA05060
+P 6000 7100
+F 0 "P5" H 6000 7050 60  0000 C CNN
+F 1 "US0119" H 6000 7150 60  0000 C CNN
+F 2 "OSHWA_Certification_Mark:OSHW_Mono_0.15_Scale" H 6000 7100 60  0001 C CNN
+F 3 "" H 6000 7100 60  0001 C CNN
+	1    6000 7100
+	1    0    0    -1
+$EndComp
 $EndSCHEMATC
