File: electronics/led_board_stack_light/led_board.kicad_pcb (KiCad board)
At the start: 2 copper layers, 55.4 x 29.5 mm, 14 parts, among them J1 CONN_01X02, J2 CONN_01X01, P1 OSHW, P2 Slot, P3 Slot, P4 Slot

Commit message: Minor updates on recent boards
Parts:
- added P5: US0119, OSHWA_Certification_Mark:OSHW_Mono_0.15_Scale, F.Cu at (142.0, 96.5)
Changed lines of the file:
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@@
-(kicad_pcb (version 4) (host pcbnew 4.0.6+dfsg1-1)
+(kicad_pcb (version 4) (host pcbnew 4.0.7)
   (general
     (links 11)
@@
     (tracks 43)
     (zones 0)
-    (modules 14)
+    (modules 15)
     (nets 9)
   )
@@
   )
   (setup
-    (last_trace_width 0.4)
+    (last_trace_width 0.25)
     (user_trace_width 0.4)
     (user_trace_width 1)
@@
     (tags "LED PLCC-2 SMD")
     (attr smd)
-    (fp_text reference D2 (at 0 -2.5 180) (layer F.SilkS)
+    (fp_text reference D2 (at 0 2.5 180) (layer F.SilkS)
       (effects (font (size 1 1) (thickness 0.15)))
     )
@@
     (fp_line (start -7.5 -1.55) (end -7.5 1.55) (layer Edge.Cuts) (width 0.15))
   )
+  (module OSHWA_Certification_Mark:OSHW_Mono_0.15_Scale (layer F.Cu)
+    (at 142 96.5)
+    (fp_text reference P5 (at 0 -2.083427) (layer F.SilkS) hide
+      (effects (font (thickness 0.04572)))
+    )
+    (fp_text value US0119 (at 0 2.7) (layer F.SilkS)
+      (effects (font (size 0.885 0.885) (thickness 0.12)))
+    )
+    (fp_poly (pts (xy -3.123406 -1.255086) (xy -3.123406 -1.128086) (xy -3.123406 1.499227) (xy -3.123406 1.626227)
+      (xy -2.996406 1.626227) (xy 2.996406 1.626227) (xy 3.123406 1.626227) (xy 3.123406 1.499227)
+      (xy 3.123406 -1.255086) (xy 2.874858 -1.255086) (xy 2.869406 1.372227) (xy -2.869406 1.372227)
+      (xy -2.869406 -1.001086) (xy 2.013479 -1.001086) (xy 2.013479 -1.255086) (xy -2.996406 -1.255086)
+      (xy -3.123406 -1.255086)) (layer F.SilkS) (width 0.00254))
+    (fp_poly (pts (xy -1.657777 0.216596) (xy -1.448425 0.216596) (xy -1.450348 0.310265) (xy -1.456115 0.397795)
+      (xy -1.465727 0.479185) (xy -1.479184 0.554436) (xy -1.496485 0.623548) (xy -1.517631 0.686521)
+      (xy -1.542621 0.743355) (xy -1.571457 0.794049) (xy -1.615719 0.852258) (xy -1.667148 0.899883)
+      (xy -1.725742 0.936924) (xy -1.791502 0.963383) (xy -1.864428 0.979258) (xy -1.944519 0.984549)
+      (xy -2.024611 0.979285) (xy -2.097537 0.963493) (xy -2.163297 0.937173) (xy -2.221891 0.900324)
+      (xy -2.273319 0.852947) (xy -2.317581 0.795041) (xy -2.346185 0.744549) (xy -2.370974 0.687824)
+      (xy -2.391949 0.624866) (xy -2.409111 0.555677) (xy -2.422459 0.480255) (xy -2.431993 0.398601)
+      (xy -2.437714 0.310715) (xy -2.43962 0.216596) (xy -2.437714 0.122695) (xy -2.431993 0.034965)
+      (xy -2.422459 -0.046596) (xy -2.409111 -0.121987) (xy -2.391949 -0.191208) (xy -2.370974 -0.254258)
+      (xy -2.346185 -0.311139) (xy -2.317581 -0.361849) (xy -2.273043 -0.420057) (xy -2.22145 -0.467681)
+      (xy -2.162801 -0.504723) (xy -2.097096 -0.531181) (xy -2.024335 -0.547057) (xy -1.944519 -0.552349)
+      (xy -1.864428 -0.547057) (xy -1.791502 -0.531181) (xy -1.725742 -0.504723) (xy -1.667148 -0.467681)
+      (xy -1.615719 -0.420057) (xy -1.571457 -0.361849) (xy -1.542621 -0.311139) (xy -1.517631 -0.254258)
+      (xy -1.496485 -0.191208) (xy -1.479184 -0.121987) (xy -1.465727 -0.046596) (xy -1.456115 0.034965)
+      (xy -1.450348 0.122695) (xy -1.448425 0.216596) (xy -1.657777 0.216596) (xy -1.659651 0.112968)
+      (xy -1.665274 0.019703) (xy -1.674645 -0.0632) (xy -1.687763 -0.13574) (xy -1.70463 -0.197917)
+      (xy -1.725245 -0.249732) (xy -1.763879 -0.310937) (xy -1.813303 -0.354655) (xy -1.873516 -0.380886)
+      (xy -1.944519 -0.38963) (xy -2.015151 -0.380886) (xy -2.07524 -0.354655) (xy -2.124788 -0.310937)
+      (xy -2.163793 -0.249732) (xy -2.184105 -0.197917) (xy -2.200724 -0.13574) (xy -2.21365 -0.0632)
+      (xy -2.222883 0.019703) (xy -2.228423 0.112968) (xy -2.230269 0.216596) (xy -2.228423 0.319922)
+      (xy -2.222883 0.412939) (xy -2.21365 0.495649) (xy -2.200724 0.568051) (xy -2.184105 0.630146)
+      (xy -2.163793 0.681932) (xy -2.124788 0.743138) (xy -2.07524 0.786856) (xy -2.015151 0.813087)
+      (xy -1.944519 0.821831) (xy -1.873516 0.813149) (xy -1.813303 0.787104) (xy -1.763879 0.743696)
+      (xy -1.725245 0.682925) (xy -1.70463 0.63111) (xy -1.687763 0.568933) (xy -1.674645 0.496394)
+      (xy -1.665274 0.413491) (xy -1.659651 0.320225) (xy -1.657777 0.216596)) (layer F.SilkS) (width 0.00254))
+    (fp_poly (pts (xy -0.329238 -0.474959) (xy -0.329238 -0.27156) (xy -0.390203 -0.307388) (xy -0.451388 -0.336823)
+      (xy -0.512793 -0.359865) (xy -0.573868 -0.3764) (xy -0.635383 -0.386322) (xy -0.697339 -0.38963)
+      (xy -0.785314 -0.382243) (xy -0.860058 -0.360084) (xy -0.921574 -0.323154) (xy -0.967325 -0.274315)
+      (xy -0.994775 -0.215115) (xy -1.003925 -0.145552) (xy -0.990531 -0.058983) (xy -0.950347 0.004268)
+      (xy -0.903604 0.036791) (xy -0.836136 0.065564) (xy -0.747941 0.090588) (xy -0.642769 0.114401)
+      (xy -0.56395 0.136071) (xy -0.49418 0.162185) (xy -0.433458 0.192745) (xy -0.381784 0.227749)
+      (xy -0.339159 0.267198) (xy -0.297488 0.324001) (xy -0.267723 0.39023) (xy -0.249863 0.465884)
+      (xy -0.243909 0.550964) (xy -0.249149 0.63149) (xy -0.264865 0.703999) (xy -0.291059 0.768491)
+      (xy -0.32773 0.824966) (xy -0.374878 0.873425) (xy -0.432029 0.91343) (xy -0.498704 0.944544)
+      (xy -0.574904 0.96677) (xy -0.660629 0.980105) (xy -0.755878 0.984549) (xy -0.825442 0.982014)
+      (xy -0.895226 0.974407) (xy -0.96523 0.961729) (xy -1.035455 0.944641) (xy -1.1059 0.922482)
+      (xy -1.176566 0.895252) (xy -1.176566 0.681932) (xy -1.101932 0.725919) (xy -1.030163 0.761307)
+      (xy -0.961261 0.788096) (xy -0.893021 0.806838) (xy -0.82456 0.818083) (xy -0.755878 0.821831)
+      (xy -0.684193 0.817614) (xy -0.620941 0.804964) (xy -0.566123 0.78388) (xy -0.519738 0.754362)
+      (xy -0.472885 0.702768) (xy -0.444773 0.639268) (xy -0.435402 0.563862) (xy -0.441907 0.495622)
+      (xy -0.46142 0.439067) (xy -0.493941 0.394198) (xy -0.541897 0.358149) (xy -0.609035 0.328052)
+      (xy -0.695355 0.303909) (xy -0.802511 0.279104) (xy -0.880537 0.258546) (xy -0.949514 0.234178)
+      (xy -1.009442 0.206) (xy -1.060321 0.174012) (xy -1.102152 0.138213) (xy -1.142956 0.087054)
+      (xy -1.172101 0.027833) (xy -1.189589 -0.03945) (xy -1.195418 -0.114794) (xy -1.190099 -0.190994)
+      (xy -1.174145 -0.260843) (xy -1.147554 -0.324343) (xy -1.110328 -0.381494) (xy -1.062464 -0.432294)
+      (xy -1.005394 -0.475513) (xy -0.941338 -0.509128) (xy -0.870298 -0.533139) (xy -0.792272 -0.547546)
+      (xy -0.707261 -0.552349) (xy -0.649384 -0.550143) (xy -0.589522 -0.543528) (xy -0.527675 -0.532505)
+      (xy -0.463735 -0.517732) (xy -0.397589 -0.49855) (xy -0.329238 -0.474959)) (layer F.SilkS) (width 0.00254))
+    (fp_poly (pts (xy 0.024973 -0.52556) (xy 0.226387 -0.52556) (xy 0.226387 0.081659) (xy 0.775067 0.081659)
+      (xy 0.775067 -0.52556) (xy 0.976481 -0.52556) (xy 0.976481 0.955776) (xy 0.775067 0.955776)
+      (xy 0.775067 0.250331) (xy 0.226387 0.250331) (xy 0.226387 0.955776) (xy 0.024973 0.955776)
+      (xy 0.024973 -0.52556)) (layer F.SilkS) (width 0.00254))
+    (fp_poly (pts (xy 1.111419 -0.52556) (xy 1.30688 -0.52556) (xy 1.448762 0.676971) (xy 1.617434 -0.118763)
+      (xy 1.826786 -0.118763) (xy 1.997442 0.678956) (xy 2.477991 -1.626227) (xy 2.673452 -1.626227)
+      (xy 2.113528 0.955776) (xy 1.92402 0.955776) (xy 1.722606 0.075706) (xy 1.522184 0.955776)
+      (xy 1.332676 0.955776) (xy 1.111419 -0.52556)) (layer F.SilkS) (width 0.00254))
+  )
   (gr_arc (start 154.99 111.5) (end 155.856 112) (angle 60) (layer Edge.Cuts) (width 0.15))
