File: electronics/square_grid_board/square_grid_board.kicad_pcb (KiCad board)
At the start: 2 copper layers, 50 x 50 mm, 12 parts, among them J1 Conn_01x03, J2 Conn_01x03, P1 OSHW, U1 5050_Serial_RGB, U2 5050_Serial_RGB, U3 5050_Serial_RGB, U4 5050_Serial_RGB, U5 5050_Serial_RGB, U6 5050_Serial_RGB, U7 5050_Serial_RGB, U8 5050_Serial_RGB, U9 5050_Serial_RGB

Commit message: Add OSHW certification to square_grid_board
Parts:
- added P2: US0120, OSHWA_Certification_Mark:OSHW_Mono_0.20_Scale, F.Cu at (145.4, 62.6)
Other:
- board text added: "(c) Google LLC"
- board text added: "+5 G D"
- board text added: "CUT OUT"
- board text added: "IN"
- board text added: "OUT"
- board text removed: "(c) Google, LLC"
Changed lines of the file:
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@@
     (area 110.814999 60.014999 160.965001 110.165001)
     (thickness 1.6)
-    (drawings 55)
+    (drawings 61)
     (tracks 179)
     (zones 0)
-    (modules 12)
+    (modules 13)
     (nets 13)
   )
@@
     (pad_to_mask_clearance 0.2)
     (aux_axis_origin 135.89 85.09)
-    (grid_origin 118.39 70.09)
+    (grid_origin 135.89 85.09)
     (visible_elements FFFFFF7F)
     (pcbplotparams
@@
       (xy -0.113933 -2.757629) (xy -0.013056 -2.757714) (xy 0 -2.757714) (xy 0.10391 -2.757652)) (layer F.SilkS) (width 0.01))
   )
-  (gr_text "(c) Google, LLC" (at 135.89 85.09) (layer B.SilkS)
-    (effects (font (size 1.5 1.5) (thickness 0.3)) (justify mirror))
+  (module OSHWA_Certification_Mark:OSHW_Mono_0.20_Scale (layer F.Cu)
+    (at 145.39 62.59)
+    (fp_text reference P2 (at 0 -2.777902) (layer F.SilkS) hide
+      (effects (font (thickness 0.06096)))
+    )
+    (fp_text value US0120 (at 0 3.6) (layer F.SilkS)
+      (effects (font (size 1.18 1.18) (thickness 0.16)))
+    )
+    (fp_poly (pts (xy -4.164542 -1.673448) (xy -4.164542 -1.504114) (xy -4.164542 1.998969) (xy -4.164542 2.168302)
+      (xy -3.995208 2.168302) (xy 3.995208 2.168302) (xy 4.164542 2.168302) (xy 4.164542 1.998969)
+      (xy 4.164542 -1.673448) (xy 3.833144 -1.673448) (xy 3.825875 1.829636) (xy -3.825875 1.829636)
+      (xy -3.825875 -1.334781) (xy 2.684639 -1.334781) (xy 2.684639 -1.673448) (xy -3.995208 -1.673448)
+      (xy -4.164542 -1.673448)) (layer F.SilkS) (width 0.00254))
+    (fp_poly (pts (xy -2.210369 0.288795) (xy -1.931234 0.288795) (xy -1.933797 0.413687) (xy -1.941487 0.530393)
+      (xy -1.954303 0.638913) (xy -1.972245 0.739248) (xy -1.995314 0.831398) (xy -2.023508 0.915362)
+      (xy -2.056829 0.99114) (xy -2.095275 1.058733) (xy -2.154293 1.136344) (xy -2.222864 1.199844)
+      (xy -2.30099 1.249233) (xy -2.38867 1.28451) (xy -2.485904 1.305677) (xy -2.592692 1.312733)
+      (xy -2.699481 1.305714) (xy -2.796716 1.284657) (xy -2.884396 1.249563) (xy -2.962521 1.200432)
+      (xy -3.031092 1.137262) (xy -3.090109 1.060055) (xy -3.128246 0.992731) (xy -3.161298 0.917098)
+      (xy -3.189266 0.833155) (xy -3.212148 0.740902) (xy -3.229945 0.64034) (xy -3.242657 0.531468)
+      (xy -3.250285 0.414286) (xy -3.252827 0.288795) (xy -3.250285 0.163594) (xy -3.242657 0.046619)
+      (xy -3.229945 -0.062128) (xy -3.212148 -0.162649) (xy -3.189266 -0.254943) (xy -3.161298 -0.339011)
+      (xy -3.128246 -0.414851) (xy -3.090109 -0.482465) (xy -3.030725 -0.560076) (xy -2.961933 -0.623575)
+      (xy -2.883734 -0.672964) (xy -2.796128 -0.708242) (xy -2.699114 -0.729409) (xy -2.592692 -0.736465)
+      (xy -2.485904 -0.729409) (xy -2.38867 -0.708242) (xy -2.30099 -0.672964) (xy -2.222864 -0.623575)
+      (xy -2.154293 -0.560076) (xy -2.095275 -0.482465) (xy -2.056829 -0.414851) (xy -2.023508 -0.339011)
+      (xy -1.995314 -0.254943) (xy -1.972245 -0.162649) (xy -1.954303 -0.062128) (xy -1.941487 0.046619)
+      (xy -1.933797 0.163594) (xy -1.931234 0.288795) (xy -2.210369 0.288795) (xy -2.212868 0.150624)
+      (xy -2.220365 0.02627) (xy -2.232859 -0.084266) (xy -2.250351 -0.180986) (xy -2.27284 -0.263889)
+      (xy -2.300327 -0.332976) (xy -2.351839 -0.414582) (xy -2.417737 -0.472873) (xy -2.498021 -0.507848)
+      (xy -2.592692 -0.519507) (xy -2.686868 -0.507848) (xy -2.766987 -0.472873) (xy -2.83305 -0.414582)
+      (xy -2.885057 -0.332976) (xy -2.91214 -0.263889) (xy -2.934299 -0.180986) (xy -2.951534 -0.084266)
+      (xy -2.963844 0.02627) (xy -2.97123 0.150624) (xy -2.973692 0.288795) (xy -2.97123 0.426562)
+      (xy -2.963844 0.550586) (xy -2.951534 0.660866) (xy -2.934299 0.757402) (xy -2.91214 0.840194)
+      (xy -2.885057 0.909243) (xy -2.83305 0.990851) (xy -2.766987 1.049142) (xy -2.686868 1.084116)
+      (xy -2.592692 1.095774) (xy -2.498021 1.084199) (xy -2.417737 1.049472) (xy -2.351839 0.991595)
+      (xy -2.300327 0.910566) (xy -2.27284 0.84148) (xy -2.250351 0.758578) (xy -2.232859 0.661858)
+      (xy -2.220365 0.551321) (xy -2.212868 0.426967) (xy -2.210369 0.288795)) (layer F.SilkS) (width 0.00254))
+    (fp_poly (pts (xy -0.438984 -0.633278) (xy -0.438984 -0.36208) (xy -0.52027 -0.409851) (xy -0.60185 -0.449097)
+      (xy -0.683723 -0.47982) (xy -0.765157 -0.501867) (xy -0.847178 -0.515096) (xy -0.929786 -0.519507)
+      (xy -1.047085 -0.509658) (xy -1.146744 -0.480112) (xy -1.228765 -0.430872) (xy -1.289766 -0.365754)
+      (xy -1.326367 -0.28682) (xy -1.338567 -0.19407) (xy -1.320708 -0.078644) (xy -1.267129 0.005691)
+      (xy -1.204806 0.049054) (xy -1.114847 0.087419) (xy -0.997254 0.120785) (xy -0.857025 0.152535)
+      (xy -0.751933 0.181428) (xy -0.658906 0.216247) (xy -0.577944 0.256993) (xy -0.509046 0.303665)
+      (xy -0.452213 0.356264) (xy -0.396651 0.432001) (xy -0.356964 0.520306) (xy -0.333151 0.621178)
+      (xy -0.325213 0.734618) (xy -0.332198 0.841986) (xy -0.353154 0.938665) (xy -0.388079 1.024654)
+      (xy -0.436973 1.099955) (xy -0.499838 1.164566) (xy -0.576038 1.217906) (xy -0.664939 1.259393)
+      (xy -0.766539 1.289026) (xy -0.880838 1.306806) (xy -1.007838 1.312733) (xy -1.100589 1.309352)
+      (xy -1.193635 1.299209) (xy -1.286973 1.282305) (xy -1.380607 1.259522) (xy -1.474534 1.229977)
+      (xy -1.568754 1.19367) (xy -1.568754 0.909243) (xy -1.469242 0.967892) (xy -1.373551 1.015076)
+      (xy -1.281682 1.050795) (xy -1.190695 1.075784) (xy -1.099413 1.090777) (xy -1.007838 1.095774)
+      (xy -0.912258 1.090152) (xy -0.827922 1.073285) (xy -0.754831 1.045173) (xy -0.692984 1.005816)
+      (xy -0.630513 0.937025) (xy -0.593031 0.852358) (xy -0.580536 0.751816) (xy -0.589209 0.660829)
+      (xy -0.615226 0.585423) (xy -0.658588 0.525597) (xy -0.722529 0.477532) (xy -0.812047 0.437403)
+      (xy -0.92714 0.405212) (xy -1.070015 0.372139) (xy -1.174049 0.344728) (xy -1.266019 0.312238)
+      (xy -1.345923 0.274667) (xy -1.413762 0.232016) (xy -1.469536 0.184285) (xy -1.523941 0.116073)
+      (xy -1.562802 0.037111) (xy -1.586118 -0.052599) (xy -1.59389 -0.153059) (xy -1.586799 -0.254658)
+      (xy -1.565527 -0.347791) (xy -1.530073 -0.432458) (xy -1.480437 -0.508658) (xy -1.416619 -0.576392)
+      (xy -1.340525 -0.634018) (xy -1.255118 -0.678838) (xy -1.160397 -0.710852) (xy -1.056363 -0.730061)
+      (xy -0.943015 -0.736465) (xy -0.865845 -0.733524) (xy -0.786029 -0.724705) (xy -0.703567 -0.710007)
+      (xy -0.618313 -0.690309) (xy -0.530119 -0.664733) (xy -0.438984 -0.633278)) (layer F.SilkS) (width 0.00254))
+    (fp_poly (pts (xy 0.033298 -0.700747) (xy 0.30185 -0.700747) (xy 0.30185 0.108878) (xy 1.033423 0.108878)
+      (xy 1.033423 -0.700747) (xy 1.301975 -0.700747) (xy 1.301975 1.274368) (xy 1.033423 1.274368)
+      (xy 1.033423 0.333774) (xy 0.30185 0.333774) (xy 0.30185 1.274368) (xy 0.033298 1.274368)
+      (xy 0.033298 -0.700747)) (layer F.SilkS) (width 0.00254))
+    (fp_poly (pts (xy 1.481891 -0.700747) (xy 1.742506 -0.700747) (xy 1.931683 0.902628) (xy 2.156579 -0.158351)
+      (xy 2.435714 -0.158351) (xy 2.663256 0.905274) (xy 3.303989 -2.168302) (xy 3.564603 -2.168302)
+      (xy 2.818037 1.274368) (xy 2.56536 1.274368) (xy 2.296808 0.100941) (xy 2.029579 1.274368)
+      (xy 1.776902 1.274368) (xy 1.481891 -0.700747)) (layer F.SilkS) (width 0.00254))
+  )
+  (gr_text "CUT OUT" (at 135.89 95.09) (layer F.SilkS)
+    (effects (font (size 1.5 1.5) (thickness 0.3)))
+  )
+  (gr_text "CUT OUT" (at 135.89 75.09) (layer F.SilkS)
+    (effects (font (size 1.5 1.5) (thickness 0.3)))
+  )
+  (gr_text "+5 G D" (at 112.39 75.09 90) (layer B.SilkS)
+    (effects (font (size 1.2 1.2) (thickness 0.3)) (justify mirror))
+  )
+  (gr_text OUT (at 116.89 95.09 90) (layer F.SilkS)
+    (effects (font (size 1 1) (thickness 0.25)))
+  )
+  (gr_text IN (at 116.89 75.09 90) (layer F.SilkS)
+    (effects (font (size 1 1) (thickness 0.25)))
+  )
+  (gr_text "+5 G D" (at 112.39 95.09 90) (layer B.SilkS)
+    (effects (font (size 1.2 1.2) (thickness 0.3)) (justify mirror))
+  )
+  (gr_text "(c) Google LLC" (at 145.89 107.59) (layer F.SilkS)
+    (effects (font (size 1.2 1.2) (thickness 0.3)))
   )
   (gr_line (start 140.39 67.09) (end 138.39 69.09) (angle 90) (layer Edge.Cuts) (width 0.15))
@@
   (gr_line (start 117.89 69.59) (end 120.39 67.09) (angle 90) (layer Edge.Cuts) (width 0.15))
   (gr_line (start 117.89 80.59) (end 117.89 69.59) (angle 90) (layer Edge.Cuts) (width 0.15))
-  (gr_text CC-BY (at 146.39 106.59) (layer F.SilkS)
-    (effects (font (size 1.5 1.5) (thickness 0.3)))
+  (gr_text CC-BY (at 146.39 105.09) (layer F.SilkS)
+    (effects (font (size 1.2 1.2) (thickness 0.3)))
   )
   (gr_text "github.com/google/makerspace-partsbin\n  electronics/square_grid_board" (at 135.89 105.59) (layer B.SilkS)
