File: electronics/square_grid_board/square_grid_board.sch (KiCad schematic (older format))
At the start: 12 parts, among them J1 Conn_01x03, J2 Conn_01x03, P1 OSHW, U1 5050_Serial_RGB, U2 5050_Serial_RGB, U3 5050_Serial_RGB, U4 5050_Serial_RGB, U5 5050_Serial_RGB, U6 5050_Serial_RGB, U7 5050_Serial_RGB, U8 5050_Serial_RGB, U9 5050_Serial_RGB

Commit message: Add OSHW certification to square_grid_board
Parts:
- added P2: US0120, OSHWA_Certification_Mark:OSHW_Mono_0.20_Scale, symbol SYMBOL
Other:
- moved on the sheet: P1
Changed lines of the file:
@@
 L SYMBOL P1
 U 1 1 5A9EFB61
+P 6600 6700
+F 0 "P1" H 6600 6650 60  0000 C CNN
+F 1 "OSHW" H 6600 6750 60  0000 C CNN
+F 2 "Symbols:OSHW-Logo2_7.3x6mm_SilkScreen" H 6600 6700 60  0001 C CNN
+F 3 "" H 6600 6700 60  0001 C CNN
+	1    6600 6700
+	1    0    0    -1
+$EndComp
+$Comp
+L SYMBOL P2
+U 1 1 5AA0336B
 P 6600 7100
-F 0 "P1" H 6600 7050 60  0000 C CNN
-F 1 "OSHW" H 6600 7150 60  0000 C CNN
-F 2 "Symbols:OSHW-Logo2_7.3x6mm_SilkScreen" H 6600 7100 60  0001 C CNN
+F 0 "P2" H 6600 7050 60  0000 C CNN
+F 1 "US0120" H 6600 7150 60  0000 C CNN
+F 2 "OSHWA_Certification_Mark:OSHW_Mono_0.20_Scale" H 6600 7100 60  0001 C CNN
 F 3 "" H 6600 7100 60  0001 C CNN
 	1    6600 7100
